File: docs/hardware/schematic/PicAmpControl.kicad_sch (KiCad schematic)
At the start: 85 parts, among them J1 Conn_01x04, J10 Conn_01x02, J11 Conn_01x01, J2 Conn_01x06, J3 Conn_01x02, J4 Conn_01x02, J5 Conn_01x03, J6 Conn_01x01, J7 Conn_01x03, J8 Conn_01x02, J9 Conn_01x02, Q1 IRLZ44N, Q2 2N3904, Q3 2N3904, Q4 2N3904, Q5 2N3904, Q6 2N3904, SW1 SW_PUSH, SW2 SW_PUSH, U1 PIC16F18855-I/SP, U10 BAT54S, U11 BAT54S, U2 PC817, U3 BAT54S, U4 BAT54S, U5 BAT54S, U6 BAT54S, U7 BAT54S, U8 BAT54S, U9 BAT54S

Commit message: Add LM7805 12V to 5V linear regulator with C1 330nF and C2 100nF decoupling capacitors to schematic and netlist
Parts:
- added C1: 330nF, Capacitor_THT:C_Disc_D3.0mm_W2.0mm_P2.50mm, symbol Device:C
- added C2: 100nF, Capacitor_THT:C_Disc_D3.0mm_W2.0mm_P2.50mm, symbol Device:C
- added U12: LM7805_TO220, Package_TO_SOT_THT:TO-220-3_Vertical, symbol Regulator_Linear:LM7805_TO220
Connections:
- net +12V_RAIL: now also C10.2, C11.2, C12.2, C13.2, C14.2, C15.2, C16.2, C3.1, C3.2, C4.1, C4.2, C5.1, C5.2, C6.2, C7.2, C8.2, C9.2, D1.1 (K), D2.1 (K), D2.2 (A), D3.1 (K), D4.1 (K), D5.1 (K), D5.2 (A), D6.1 (K), D6.2 (A), D7.1 (K), D7.2 (A), J1.1 (Pin_1), J1.2 (Pin_2), J10.2 (Pin_2), J2.5 (Pin_5), J2.6 (Pin_6), J3.1 (Pin_1), J5.1 (Pin_1), J6.1 (Pin_1), J7.1 (Pin_1), J7.2 (Pin_2), J7.3 (Pin_3), Q1.1 (G), Q1.3 (S), Q2.1 (E), Q2.3 (C), Q3.1 (E), Q4.1 (E), Q5.1 (E), Q5.3 (C), Q6.1 (E), R1.1, R1.2, R10.2, R12.2, R14.2, R16.2, R18.1, R2.2, R27.2, R3.1, R3.2, R30.2, R31.1, R32.1, R33.1, R34.1, R34.2, R4.1, R4.2, R5.1, R6.1, R8.2, SW1.1, SW1.2, SW2.1, SW2.2, U1.1 (MCLR/VPP), U1.11 (VDD), U1.20 (VSS), U1.21 (RC0), U1.8 (VSS), U10.1 (A1), U10.2 (K2), U11.1 (A1), U11.2 (K2), U2.3 (E), U3.1 (A1), U3.2 (K2), U4.1 (A1), U4.2 (K2), U5.1 (A1), U5.2 (K2), U6.1 (A1), U6.2 (K2), U7.1 (A1), U7.2 (K2), U8.1 (A1), U8.2 (K2), U9.1 (A1), U9.2 (K2), C1.1, C1.2, C2.1, C2.2
- net CURRENT: now also C10.1, C11.1, C12.1, C13.1, C7.1, C8.1, C9.1, R20.2, R21.2, R22.2, R23.2, R24.2, R25.2, R26.2, U1.13 (RB1/AN9), U1.14 (RB2/AN10), U1.16 (RB4), U1.3 (RA1/AN1), U1.4 (RA2/AN2), U1.5 (RA3/AN3), U1.7 (RA5/AN5), U10.3 (K1A2), U4.3 (K1A2), U5.3 (K1A2), U6.3 (K1A2), U7.3 (K1A2), U8.3 (K1A2), U9.3 (K1A2)
- net DRAIN_PEAK: now also C14.1, R31.2, U1.15 (RB3/AN11), U11.3 (K1A2)
- net FAN_PWM: now also R2.1, U1.17 (RB5)
- net LCD_SCL: now also J1.3 (Pin_3), J1.4 (Pin_4), R5.2, R6.2, U1.24 (RC3/SCL), U1.25 (RC4/SDA)
- net MENU_ADJUST: now also C15.1, R32.2, U1.12 (RB0)
- net MENU_NEXT: now also C16.1, R33.2, U1.23 (RC2)
- net SWR1_FWD: now also C6.1, R19.2, U1.2 (RA0/AN0), U3.3 (K1A2)
- net TX_BIAS_BASE: now reaches Q4.2 (B)
- net TX_BIAS_BASE: now also R11.2, R12.1
- net TX_BIAS: now reaches Q4.3 (C)
- net TX_BIAS: now also D3.2 (A), D4.2 (A), J5.2 (Pin_2), J5.3 (Pin_3), Q3.3 (C)
- net PTT_ANODE: now reaches U2.1 (A)
- net PTT_ANODE: now also R17.2
- net PTT_CATHODE: now reaches U2.2 (K)
- net PTT_CATHODE: now also J4.2 (Pin_2)
- net PTT_COLLECTOR: now reaches U2.4 (C)
- net PTT_COLLECTOR: now also R18.2, R27.1
- net COMP_RESET: now reaches R9.1
- net COMP_RESET: now also J2.4 (Pin_4), Q6.3 (C), R11.1, R13.1, R15.1, R7.1, U1.19 (RB7), U1.22 (RC1), U1.26 (RC5), U1.27 (RC6), U1.28 (RC7)
- net TX_VCC_BASE: now reaches R9.2
- net TX_VCC_BASE: now also Q3.2 (B), R10.1
- net PTT_EXT: now reaches J4.1 (Pin_1)
- net PTT_EXT: now also R17.1
- net SWR1_REF_RAW: now reaches R20.1
- net SWR1_REF_RAW: now also J8.2 (Pin_2)
- net COMP_RESET_BASE: now reaches Q6.2 (B)
- net COMP_RESET_BASE: now also R15.2, R16.1
- net TEMP_RAW: now reaches J10.1 (Pin_1)
- net TEMP_RAW: now also R23.1
- net SWR2_FWD_RAW: now reaches R21.1
- net SWR2_FWD_RAW: now also J9.1 (Pin_1)
- net TX_BASE: now reaches Q2.2 (B)
- net TX_BASE: now also R7.2, R8.1
- net SWR1_FWD_RAW: now reaches J8.1 (Pin_1)
- net SWR1_FWD_RAW: now also R19.1
- net TRIP_BASE: now reaches R14.1
- net TRIP_BASE: now also Q5.2 (B), R13.2
- net SWR2_REF_RAW: now reaches J9.2 (Pin_2)
- net SWR2_REF_RAW: now also R22.1
- net OC_FAULT_RAW: now reaches R25.1
- net OC_FAULT_RAW: now also J2.1 (Pin_1), J2.3 (Pin_3), R26.1
- net FAN_DRAIN: now reaches D1.2 (A)
- net FAN_DRAIN: now also J3.2 (Pin_2), Q1.2 (D)
- net DRAIN_MID1: now reaches R29.1
- net DRAIN_MID1: now also R28.2
- net DRAIN_MID2: now reaches R29.2
- net DRAIN_MID2: now also R30.1
- net CURRENT_RAW: now reaches J11.1 (Pin_1)
- net CURRENT_RAW: now also R24.1
- net DRAIN_HV: now reaches R28.1
- net DRAIN_HV: now also J2.2 (Pin_2)
Other:
- moved on the sheet: C10, C11, C12, C13, C14, C15, C16, C3, C4, C5, C6, C7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
