File: docs/hardware/schematic/PicAmpControl.kicad_pcb (KiCad board)
At the start: 2 copper layers, 85 parts, among them J1 Conn_01x04, J10 Conn_01x02, J11 Conn_01x01, J2 Conn_01x06, J3 Conn_01x02, J4 Conn_01x02, J5 Conn_01x03, J6 Conn_01x01, J7 Conn_01x03, J8 Conn_01x02, J9 Conn_01x02, Q1 IRLZ44N, Q2 2N3904, Q3 2N3904, Q4 2N3904, Q5 2N3904, Q6 2N3904, SW1 SW_PUSH, SW2 SW_PUSH, U1 PIC16F18855-I/SP, U10 BAT54S, U11 BAT54S, U2 PC817, U3 BAT54S, U4 BAT54S, U5 BAT54S, U6 BAT54S, U7 BAT54S, U8 BAT54S, U9 BAT54S

Commit message: Add LM7805 12V to 5V linear regulator with C1 330nF and C2 100nF decoupling capacitors to schematic and netlist
Parts:
- added C1: 330nF, Capacitor_THT:C_Disc_D3.0mm_W2.0mm_P2.50mm, F.Cu at (100.0, 50.0)
- added C2: 100nF, Capacitor_THT:C_Disc_D3.0mm_W2.0mm_P2.50mm, F.Cu at (125.0, 50.0)
- added U12: LM7805_TO220, Package_TO_SOT_THT:TO-220-3_Vertical, F.Cu at (75.0, 50.0)
- moved C13 126.6 mm to (50.0, 150.0)
- moved C14 126.6 mm to (75.0, 150.0)
- moved C15 126.6 mm to (100.0, 150.0)
- moved C6 126.6 mm to (75.0, 130.0)
- moved C7 126.6 mm to (100.0, 130.0)
- moved D6 126.6 mm to (50.0, 170.0)
- moved J4 126.6 mm to (50.0, 250.0)
- moved J5 126.6 mm to (75.0, 250.0)
- moved J6 126.6 mm to (100.0, 250.0)
- moved Q5 126.6 mm to (50.0, 190.0)
- moved Q6 126.6 mm to (75.0, 190.0)
- moved R13 126.6 mm to (50.0, 210.0)
- moved R14 126.6 mm to (75.0, 210.0)
- moved R15 126.6 mm to (100.0, 210.0)
- moved R17 126.6 mm to (75.0, 70.0)
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
Commit message: Fix BAT54S designators and clean up schematic wire routing
Parts:
- removed U10, U11, U3, U4, U5, U6, U7, U8, U9: BAT54S, Package_TO_SOT_SMD:SOT-23
- added D10: BAT54S, Package_TO_SOT_SMD:SOT-23, F.Cu at (225.0, 70.0)
- added D11: BAT54S, Package_TO_SOT_SMD:SOT-23, F.Cu at (50.0, 90.0)
- added D12: BAT54S, Package_TO_SOT_SMD:SOT-23, F.Cu at (75.0, 90.0)
- added D13: BAT54S, Package_TO_SOT_SMD:SOT-23, F.Cu at (100.0, 90.0)
- added D14: BAT54S, Package_TO_SOT_SMD:SOT-23, F.Cu at (125.0, 90.0)
- added D15: BAT54S, Package_TO_SOT_SMD:SOT-23, F.Cu at (150.0, 90.0)
- added D16: BAT54S, Package_TO_SOT_SMD:SOT-23, F.Cu at (175.0, 90.0)
- added D8: BAT54S, Package_TO_SOT_SMD:SOT-23, F.Cu at (175.0, 70.0)
- added D9: BAT54S, Package_TO_SOT_SMD:SOT-23, F.Cu at (200.0, 70.0)
Changed lines of the file:
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@@
   )
   (footprint "Package_TO_SOT_SMD:SOT-23" (layer "F.Cu") (at 175.00 70.00) (unit 1)
-    (property "Reference" "U3" (at 175.00 66.00 0) (layer "F.SilkS") (effects (font (size 1 1) (thickness 0.15))))
+    (property "Reference" "D8" (at 175.00 66.00 0) (layer "F.SilkS") (effects (font (size 1 1) (thickness 0.15))))
     (property "Value" "BAT54S" (at 175.00 74.00 0) (layer "F.Fab") (effects (font (size 1 1) (thickness 0.15))))
   )
   (footprint "Package_TO_SOT_SMD:SOT-23" (layer "F.Cu") (at 200.00 70.00) (unit 1)
-    (property "Reference" "U4" (at 200.00 66.00 0) (layer "F.SilkS") (effects (font (size 1 1) (thickness 0.15))))
+    (property "Reference" "D9" (at 200.00 66.00 0) (layer "F.SilkS") (effects (font (size 1 1) (thickness 0.15))))
     (property "Value" "BAT54S" (at 200.00 74.00 0) (layer "F.Fab") (effects (font (size 1 1) (thickness 0.15))))
   )
   (footprint "Package_TO_SOT_SMD:SOT-23" (layer "F.Cu") (at 225.00 70.00) (unit 1)
-    (property "Reference" "U5" (at 225.00 66.00 0) (layer "F.SilkS") (effects (font (size 1 1) (thickness 0.15))))
+    (property "Reference" "D10" (at 225.00 66.00 0) (layer "F.SilkS") (effects (font (size 1 1) (thickness 0.15))))
     (property "Value" "BAT54S" (at 225.00 74.00 0) (layer "F.Fab") (effects (font (size 1 1) (thickness 0.15))))
   )
   (footprint "Package_TO_SOT_SMD:SOT-23" (layer "F.Cu") (at 50.00 90.00) (unit 1)
-    (property "Reference" "U6" (at 50.00 86.00 0) (layer "F.SilkS") (effects (font (size 1 1) (thickness 0.15))))
+    (property "Reference" "D11" (at 50.00 86.00 0) (layer "F.SilkS") (effects (font (size 1 1) (thickness 0.15))))
     (property "Value" "BAT54S" (at 50.00 94.00 0) (layer "F.Fab") (effects (font (size 1 1) (thickness 0.15))))
   )
   (footprint "Package_TO_SOT_SMD:SOT-23" (layer "F.Cu") (at 75.00 90.00) (unit 1)
-    (property "Reference" "U7" (at 75.00 86.00 0) (layer "F.SilkS") (effects (font (size 1 1) (thickness 0.15))))
+    (property "Reference" "D12" (at 75.00 86.00 0) (layer "F.SilkS") (effects (font (size 1 1) (thickness 0.15))))
     (property "Value" "BAT54S" (at 75.00 94.00 0) (layer "F.Fab") (effects (font (size 1 1) (thickness 0.15))))
   )
   (footprint "Package_TO_SOT_SMD:SOT-23" (layer "F.Cu") (at 100.00 90.00) (unit 1)
-    (property "Reference" "U8" (at 100.00 86.00 0) (layer "F.SilkS") (effects (font (size 1 1) (thickness 0.15))))
+    (property "Reference" "D13" (at 100.00 86.00 0) (layer "F.SilkS") (effects (font (size 1 1) (thickness 0.15))))
     (property "Value" "BAT54S" (at 100.00 94.00 0) (layer "F.Fab") (effects (font (size 1 1) (thickness 0.15))))
   )
   (footprint "Package_TO_SOT_SMD:SOT-23" (layer "F.Cu") (at 125.00 90.00) (unit 1)
-    (property "Reference" "U9" (at 125.00 86.00 0) (layer "F.SilkS") (effects (font (size 1 1) (thickness 0.15))))
+    (property "Reference" "D14" (at 125.00 86.00 0) (layer "F.SilkS") (effects (font (size 1 1) (thickness 0.15))))
     (property "Value" "BAT54S" (at 125.00 94.00 0) (layer "F.Fab") (effects (font (size 1 1) (thickness 0.15))))
   )
   (footprint "Package_TO_SOT_SMD:SOT-23" (layer "F.Cu") (at 150.00 90.00) (unit 1)
-    (property "Reference" "U10" (at 150.00 86.00 0) (layer "F.SilkS") (effects (font (size 1 1) (thickness 0.15))))
+    (property "Reference" "D15" (at 150.00 86.00 0) (layer "F.SilkS") (effects (font (size 1 1) (thickness 0.15))))
     (property "Value" "BAT54S" (at 150.00 94.00 0) (layer "F.Fab") (effects (font (size 1 1) (thickness 0.15))))
   )
   (footprint "Package_TO_SOT_SMD:SOT-23" (layer "F.Cu") (at 175.00 90.00) (unit 1)
-    (property "Reference" "U11" (at 175.00 86.00 0) (layer "F.SilkS") (effects (font (size 1 1) (thickness 0.15))))
+    (property "Reference" "D16" (at 175.00 86.00 0) (layer "F.SilkS") (effects (font (size 1 1) (thickness 0.15))))
     (property "Value" "BAT54S" (at 175.00 94.00 0) (layer "F.Fab") (effects (font (size 1 1) (thickness 0.15))))
   )
