File: docs/hardware/lpf_band_decoder.kicad_sch (KiCad schematic)
At the start: 0 parts

Commit message: Complete LPF relay driver schematic
Parts:
- added C1: 100nF MCU, symbol Custom:Decoupling_C
- added C2: 100nF DEC, symbol Custom:Decoupling_C
- added C3: 100nF DRV, symbol Custom:Decoupling_C
- added D1, D2, D3, D4, D5, D6, D7: 1N4007, symbol Custom:Flyback_Diode
- added J1: +12V, symbol Custom:Power_12V
- added K1: 160m, symbol Custom:Relay_Coil
- added K2: 80m, symbol Custom:Relay_Coil
- added K3: 40m, symbol Custom:Relay_Coil
- added K4: 20m, symbol Custom:Relay_Coil
- added K5: 15m, symbol Custom:Relay_Coil
- added K6: 10m, symbol Custom:Relay_Coil
- added K7: 6m, symbol Custom:Relay_Coil
- added U1: PIC16F18855, symbol Custom:MCU_Bus
- added U2: 74HC4514, symbol Custom:Decoder_74HC4514
- added U3: ULN2803A, symbol Custom:Driver_ULN2803A
Connections:
- new net: D7.1 (A), D7.2 (K), K7.1 (COIL+), K7.2 (COIL-), U3.18 (OUT1)
- new net: D3.1 (A), D3.2 (K), K3.1 (COIL+), K3.2 (COIL-), U3.14 (OUT5)
- new net: D2.1 (A), D2.2 (K), K2.1 (COIL+), K2.2 (COIL-), U3.13 (OUT6)
- new net: D1.1 (A), D1.2 (K), K1.1 (COIL+), K1.2 (COIL-), U3.12 (OUT7)
- new net: D4.1 (A), D4.2 (K), K4.1 (COIL+), K4.2 (COIL-), U3.15 (OUT4)
- new net: D5.1 (A), D5.2 (K), K5.1 (COIL+), K5.2 (COIL-), U3.16 (OUT3)
- new net: D6.1 (A), D6.2 (K), K6.1 (COIL+), K6.2 (COIL-), U3.17 (OUT2)
- new net: U2.6 (Y1), U3.3 (IN3)
- new net: U2.7 (Y2), U3.4 (IN4)
- new net: U2.8 (Y3), U3.5 (IN5)
- new net: U1.1 (B0), U2.1 (A0)
- new net: U1.2 (B1), U2.2 (A1)
- new net: U1.3 (B2), U2.3 (A2)
- new net: U1.4 (B3), U2.4 (A3)
- new net +5V: C1.1 (+5V), C2.1 (+5V), C3.1 (+5V)
- new net DEC_10M: U2.5 (Y0), U2.9 (Y4), U3.1 (IN1), U3.6 (IN6), U3.7 (IN7)
- new net GND: C1.2 (GND), C2.2 (GND), C3.2 (GND)
Other:
- note added: "B0"
- note added: "B1"
- note added: "B2"
- note added: "B3"
- note added: "One relay energized at a time; flyback diode per coil"
- note added: "PIC B0..B3 -> 74HC4514 -> ULN2803A -> relay coil bank"
- note added: "Relay bank"
- note added: "Y1"
- note added: "Y2"
- note added: "Y3"
- note added: "Y4"
- note removed: "+12 V relay supply"
- note removed: "10m"
- note removed: "15m"
- note removed: "160m"
- note removed: "20m"
- note removed: "40m"
- note removed: "6m"
- note removed: "80m"
- note removed: "A0 B0"
- note removed: "A1 B1"
- note removed: "A2 B2"
- note removed: "A3 B3"
- note removed: "B0=RA4"
- note removed: "B1=RA6"
- note removed: "B2=RA7"
- note removed: "B3=RB6"
- note removed: "IN1..IN7"
- note removed: "LPF relay bank"
- note removed: "OUT1..OUT7"
- note removed: "flyback diodes on each relay coil"
- note removed: "logic ground common with relay ground"
