File: docs/hardware/project_schematic_package/generated/pic_amp_protection.kicad_sch (KiCad schematic)
At the start: 0 parts

Commit message: Add structured schematic generation rules
Changed lines of the file:
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@@
     (comment 4 ""))
   (sheet
-    (at 135.64 107.95)
+    (at 135.64 62.23)
     (size 25.91 17.78)
     (exclude_from_sim no)
@@
       (color 0 0 0 0.0))
     (property "Sheetname" "mcu_control1"
-      (at 135.64 107.24 0)
+      (at 135.64 61.52 0)
       (effects
         (font
@@
         (justify left bottom)))
     (property "Sheetfile" "pic_amp_protection_mcu_control1.kicad_sch"
-      (at 135.64 126.31 0)
+      (at 135.64 80.59 0)
       (effects
         (font
@@
         (justify left top))))
   (sheet
-    (at 135.38 62.23)
+    (at 135.38 107.95)
     (size 26.42 17.78)
     (exclude_from_sim no)
@@
       (color 0 0 0 0.0))
     (property "Sheetname" "band_decoder1"
-      (at 135.38 61.52 0)
+      (at 135.38 107.24 0)
       (effects
         (font
@@
         (justify left bottom)))
     (property "Sheetfile" "pic_amp_protection_band_decoder1.kicad_sch"
-      (at 135.38 80.59 0)
+      (at 135.38 126.31 0)
       (effects
         (font

Commit message: Update schematic generation work
Changed lines of the file:
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@@
         (justify left top))))
   (sheet
-    (at 135.38 107.95)
+    (at 135.38 85.09)
     (size 26.42 17.78)
     (exclude_from_sim no)
@@
       (color 0 0 0 0.0))
     (property "Sheetname" "band_decoder1"
-      (at 135.38 107.24 0)
+      (at 135.38 84.38 0)
       (effects
         (font
@@
         (justify left bottom)))
     (property "Sheetfile" "pic_amp_protection_band_decoder1.kicad_sch"
-      (at 135.38 126.31 0)
+      (at 135.38 103.45 0)
       (effects
         (font
@@
         (justify left top))))
   (sheet
-    (at 135.89 85.09)
+    (at 135.89 107.95)
     (size 25.4 17.78)
     (exclude_from_sim no)
@@
       (color 0 0 0 0.0))
     (property "Sheetname" "relay_bank1"
-      (at 135.89 84.38 0)
+      (at 135.89 107.24 0)
       (effects
         (font
@@
         (justify left bottom)))
     (property "Sheetfile" "pic_amp_protection_relay_bank1.kicad_sch"
-      (at 135.89 103.45 0)
+      (at 135.89 126.31 0)
       (effects
         (font
