File: docs/hardware/project_schematic_package/generated/pic_amp_protection_mcu_control1.kicad_sch (KiCad schematic)
At the start: 9 parts, among them J3 LCD_I2C, Q1 Q_NMOS, U1 PIC16F18855-xSO

Commit message: Add structured schematic generation rules
Connections:
- net +12V: no longer FAN1.1 (+)
- net +5V: now also C1.2, C2.2, C3.2, J3.3 (Pin_3); no longer C1.1, C2.1, C3.1, J3.1 (Pin_1)
- net GND: now also C1.1, C2.1, C3.1; no longer C1.2, C2.2, C3.2, Q1.S
- net at FAN1.2 (-): no longer Q1.D
- net BAND_B0: no longer names the net of U1.6 (RA4)
- net BAND_B1: no longer names the net of U1.10 (RA6)
- net BAND_B2: no longer names the net of U1.9 (RA7)
- net COMP_RESET: no longer names the net of U1.12 (RC1)
- net CURRENT_ADC: no longer names the net of U1.22 (RB1)
- net DRAIN_PEAK_ADC: no longer names the net of U1.24 (RB3)
- net ENCODER_A: no longer names the net of U1.13 (RC2)
- net ENCODER_B: no longer names the net of U1.21 (RB0)
- net ENCODER_SWITCH: no longer names the net of U1.27 (RB6/ICSPCLK)
- net FAN_PWM: no longer names the net of U1.26 (RB5)
- net FAN_PWM: no longer Q1.G
- removed net I2C_SCL: J3.3 (Pin_3), J3.4 (Pin_4), U1.14 (RC3), U1.15 (RC4)
- net OVERCURRENT_FAULT: no longer names the net of U1.25 (RB4)
- net OVERDRIVE_ADC: no longer names the net of U1.23 (RB2)
- net PTT_IN: no longer names the net of U1.11 (RC0)
- net SWR1_FWD_ADC: no longer names the net of U1.2 (RA0)
- net SWR1_REF_ADC: no longer names the net of U1.3 (RA1)
- net SWR2_FWD_ADC: no longer names the net of U1.4 (RA2)
- net SWR2_REF_ADC: no longer names the net of U1.5 (RA3)
- net TRIP_STATUS: no longer names the net of U1.28 (RB7/ICSPDAT)
- net TX_BIAS: no longer names the net of U1.18 (RC7)
- net TX_OUT: no longer names the net of U1.16 (RC5)
- net TX_VCC: no longer names the net of U1.17 (RC6)
Other:
- moved on the sheet: C1, C2, C3, J3, R1, RN1

Commit message: Update schematic generation work
Connections:
- net GND is gone; now on net +5V: C1.1, C2.1, C3.1, J3.2 (Pin_2), U1.19 (VSS), U1.8 (VSS)
- net +12V: now also FAN1.1 (+)
- net +5V: now also J3.1 (Pin_1), Q1.S, R1.2, RN1.2, U1.1 (RE3/~{MCLR}/VPP); no longer J3.3 (Pin_3), RN1.1
- net at J3.4 (Pin_4): now also J3.3 (Pin_3), U1.14 (RC3), U1.15 (RC4)
- net at U1.26 (RB5): now also Q1.G
- net at U1.7 (RA5): now also RN1.1; no longer RN1.2
- net at FAN1.2 (-): now also Q1.D
Other:
- moved on the sheet: C1, C2, C3, FAN1, J3, Q1, R1, RN1, U1
